File: testBoard.brd (EAGLE design)
At the start: 106.5 x 56.5 mm, 19 parts, among them IC1 AM3358BZCZ100, IC3 LM317MABDT, J1 1040310811

Commit message: syncing edit
Parts:
- removed R5: 10ohm, rcl:R0805W
- added IC5: REG1117, burr-brown:SOT223
- added JP1: (no value), pinhead:1X02
- added U$2: 4_PIN_RESISTIVE_TOUCH, 4_pin_resistive_touch_pins:4_PIN_RESISTIVE_TOUCH_CONNECTOR
- R3, R4: value 10ohm -> 100ohm
- moved C1 85.1 mm to (27.6, 6.38), flipped to the bottom, turned to 270 degrees
- moved R1 83.4 mm to (29.5, 14.6), flipped to the bottom, turned to 180 degrees
- moved R4 74.3 mm to (33.5, 13.7), turned to 270 degrees
- moved C2 71.1 mm to (24.4, 14.0), turned to 90 degrees
- moved C3 70.6 mm to (29.4, 14.7)
- moved R3 66.5 mm to (29.1, 11.3), turned to 180 degrees
- moved J1 49.3 mm to (81.8, 42.8), flipped to the top, turned to 0 degrees
- moved D3 10.8 mm to (24.3, 9.06)
- moved IC3 9.25 mm to (35.6, 6.76), flipped to the bottom
- moved R2 6.88 mm to (29.2, 11.3)
- moved D2 4.82 mm to (24.3, 8.99), flipped to the bottom, turned to 270 degrees
- moved DISPLAY 0.87 mm to (13.5, 23.2)
Connections:
- removed net N$47: J1.4
- removed net N$48: J1.6
- removed net N$49: J1.8
- removed net N$5: J1.2
- removed net N$52: R4.2, R5.2
- removed net N$53: R1.1, R4.1
- removed net N$54: R3.1
- removed net N$55: R1.2, R3.2
- removed net N$59: J1.1
- removed net N$61: J1.3
- removed net N$62: J1.5
- removed net N$63: J1.7
- removed net N$64: IC1.G15
- removed net N$65: IC1.G16
- removed net N$66: IC1.G17
- removed net N$67: IC1.G18
- removed net VO: C2.1, D2.C, D3.A, IC3.4
- new net N$37: IC3.4, R1.2
- new net N$9: IC3.1
- new net SD_CLK: IC1.G17, J1.5
- new net SD_CMD: IC1.G18, J1.3
- new net SD_D0: IC1.G16, J1.7
- new net SD_D1: IC1.G15, J1.8
- new net SD_D2: IC1.F18, J1.1
- new net SD_D3: IC1.F17, J1.2
- new net VIN_5: C2.1, D2.C, D3.A
- net GND: now also IC5.1, J1.6, JP1.1, R3.1, R4.1
- net N$50: now also R1.1, R3.2, R4.2; no longer IC3.1, R5.1
- net VIN: now also IC5.3, JP1.2
- net VIN_3.3: now also IC5.2, J1.4
Routing:
- net GND: track 1.60 -> 37.6 mm, vias 3 -> 9
- net VIN: track 0.00 -> 25.2 mm
- net SD_D2: track 0.00 -> 22.6 mm, vias 0 -> 2
- net SD_D3: track 0.00 -> 22.4 mm, vias 0 -> 2
- net N$50: track 0.00 -> 21.1 mm, vias 0 -> 2
- net SD_CMD: track 0.00 -> 20.4 mm
- net SD_D1: track 0.00 -> 19.8 mm, vias 0 -> 2
- net SD_CLK: track 0.00 -> 19.0 mm
- net SD_D0: track 0.00 -> 18.9 mm, vias 0 -> 2
- net N$37: track 0.00 -> 11.1 mm
- net VIN_5: track 0.00 -> 5.93 mm, vias 0 -> 1
Other:
- board size 106.5 x 56.5 mm -> 106.5 x 56 mm
- board text added: "+"
- board text added: "-"
- board text added: "1"
- board text added: "2"
- board text added: "3"
- board text added: "4"
- board text added: "Made by Samarth fenrir-so.tech Ref -> aq003_cortexA8/testBoard PROTOTYE 001"
- board text added: "SD Card"
- board text added: "microphone"
- board text added: "power"
- board text added: "touch connector"

Commit message: syncing edit
Connections:
- removed net N$45: IC1.L1
Changed lines of the file:
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@@
 <wire x1="46.37926875" y1="37.155" x2="45.405" y2="37.155" width="0.1" layer="1"/>
-</signal>
-<signal name="N$45">
-<contactref element="IC1" pad="L1"/>
 </signal>
 <signal name="DDR_D9">

Commit message: syncing edit
Parts:
- added C10, C7: 1uf, rcl:C0805
- added C11, C8: 10uf, rcl:C0805
- added C6, C9: 0.01uf, rcl:C0805
- added D1, D4, D5, D6: 1n4002, diode:DO-214AC
- added DISPLAY_POWER, PS2, PS3, PS4: (no value), pinhead:1X02
- added IC2, IC4: LM317MABDT, v-reg:DPACK
- added R10, R13, R16, R17, R5, R9: 10ohm, rcl:R0805W
- added R11, R8: 1kohm, rcl:R0805W
- added R12: 3.3kohm, rcl:R0805W
- added R14, R19: 470ohm, rcl:R0805W
- added R15: 100ohm, rcl:R0805W
- renumbered JP1 to PS1
Connections:
- new net DISPLAY_POWER: DISPLAY.4, DISPLAY_POWER.2
- new net N$38: R3.2, R4.2
- new net N$40: R12.1, R5.1
- new net N$41: R2.1, R3.1
- new net N$42: C8.1, D1.A, IC2.1, R11.1, R12.2, R8.1
- new net N$43: R5.2, R9.2
- new net N$44: R10.1, R9.1
- new net N$45: R10.2, R13.2
- new net N$46: C11.1, D5.A, IC4.1, R15.1, R19.2
- new net N$47: R14.1, R19.1
- new net N$48: R14.2, R16.2
- new net N$49: R16.1, R17.2
- new net VIN_1: D5.C, D6.A, IC4.4, R15.2
- new net VIN_12: C10.1
- new net VIN_9.6: C7.1
- net GND: now also C10.2, C11.2, C6.2, C7.2, C8.2, C9.2, PS2.1, PS3.1, PS4.1, R13.1, R17.1; no longer R2.1, R3.1
- net N$50: no longer R1.1, R2.2, R3.2, R4.2
- net N$9: now also R1.1, R2.2
- net VIN: now also C6.1, C9.1, D4.C, D6.C, IC2.3, IC4.3, PS2.2, PS3.2, PS4.2
- net VIN_3.3: now also DISPLAY_POWER.1; no longer DISPLAY.4
- net VIN_5: now also D1.C, D4.A, IC2.4, R11.2, R8.2
Routing:
- net N$50: track 21.1 -> 16.3 mm
- net GND: track 37.6 -> 35.5 mm, vias 9 -> 8
- net N$3: track 10.6 -> 9.53 mm
