File: testBoard.brd (EAGLE design)
At the start: 106.5 x 56 mm, 48 parts, among them IC1 AM3358BZCZ100, IC2 LM317MABDT, IC3 LM317MABDT, IC4 LM317MABDT, J1 1040310811, J2 54104-4031, J3 200529-0040

Commit message: checkpoint
Parts:
- removed R3, R4: 100ohm, rcl:R0805W
- added C12, C15, C18: 0.01uf, rcl:C0805
- added C13, C16, C19: 1uf, rcl:C0805
- added C14, C17, C20: 10uf, rcl:C0805
- added D10, D11, D12, D7, D8, D9: 1n4002, diode:DO-214AC
- added IC5, IC6, IC7: LM317MABDT, v-reg:DPACK
- added J4: M50-3610542R, M50-3610542R:M503610542
- added R18, R21, R23: 246ohm, rcl:R0805W
- added R20, R22, R24: 150ohm, rcl:R0805W
- R2: value 100ohm -> 30ohm
- moved C9 141.5 mm to (25.0, 37.8), flipped to the bottom, turned to 90 degrees
- moved C11 117.0 mm to (24.0, 14.4), flipped to the bottom, turned to 180 degrees
- moved R19 107.1 mm to (23.9, 11.8), flipped to the bottom
- moved R17 106.6 mm to (23.9, 5.10), flipped to the bottom, turned to 180 degrees
- moved C10 104.7 mm to (23.8, 2.90), flipped to the bottom
- moved R13 102.4 mm to (39.1, 20.7), flipped to the bottom, turned to 180 degrees
- moved R15 102.0 mm to (23.6, 5.40)
- moved R16 99.7 mm to (23.8, 9.50), flipped to the bottom
- moved R14 99.6 mm to (23.8, 7.20), flipped to the bottom
- moved IC4 99.4 mm to (26.4, 13.4)
- moved D6 92.2 mm to (26.4, 17.5), flipped to the bottom
- moved R12 89.4 mm to (33.8, 14.7), flipped to the bottom
- moved R11 85.2 mm to (37.7, 12.6), flipped to the bottom, turned to 270 degrees
- moved R10 84.9 mm to (43.3, 19.1), flipped to the bottom, turned to 90 degrees
- moved D5 79.9 mm to (24.6, 2.80), turned to 180 degrees
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Connections:
- removed net N$38: R3.2, R4.2
- removed net N$41: R2.1, R3.1
- removed net N$50: C3.1, D2.A
- removed net VIN_1: D5.C, D6.A, IC4.4, R15.2
- new net JTAG_TCK: IC1.A12, J4.4
- new net JTAG_TDI: IC1.B11, J4.8
- new net JTAG_TDO: IC1.A11, J4.6
- new net JTAG_TEST_RESET_NTRST: IC1.B10, J4.9
- new net JTAG_TMS: IC1.C11, J4.2
- new net N$10: C20.1, D11.A, IC7.1, R23.2, R24.1
- new net N$6: C14.1, D7.A, IC5.1, R18.2, R20.1
- new net N$7: C17.1, D9.A, IC6.1, R21.2, R22.1
- new net NRESET_IN_OUT_AM3358: IC1.A10, J4.10
- net GND: now also C12.2, C13.2, C14.2, C15.2, C16.2, C17.2, C18.2, C19.2, C20.2, J4.3, J4.5, R18.1, R2.1, R21.1, R23.1; no longer R4.1
- net N$9: now also C3.1, D2.A
- net VIN: now also C12.1, C15.1, C18.1, D10.C, D12.C, D8.C, IC5.3, IC6.3, IC7.3
- net VIN_12: now also D5.C, D6.A, IC4.4, R15.2
- net VIN_3.3: now also C13.1, C16.1, C19.1, D10.A, D11.C, D12.A, D7.C, D8.A, D9.C, IC5.4, IC6.4, IC7.4, J4.1, R20.2, R22.2, R24.2
- net VIN_5: now also IC3.4, R1.2; no longer D1.C, D4.A, IC2.4, R11.2, R8.2
- net VIN_9.6: now also D1.C, D4.A, IC2.4, R11.2, R8.2
Routing:
- net VIN: track 0.72 -> 120.2 mm, vias 0 -> 6
- net VIN_3.3: track 0.00 -> 83.4 mm, vias 0 -> 4
- net VIN_9.6: track 0.00 -> 69.7 mm, vias 0 -> 2
- net LCD_DATA18: track 0.00 -> 60.1 mm, vias 0 -> 2
- net LCD_DATA0: track 0.00 -> 59.7 mm
- net LCD_DATA1: track 0.00 -> 59.0 mm, vias 0 -> 2
- net LCD_DATA21: track 0.00 -> 58.7 mm, vias 0 -> 2
- net LCD_DATA16: track 0.00 -> 58.6 mm, vias 0 -> 2
- net LCD_DATA2: track 0.00 -> 57.6 mm, vias 0 -> 2
- net LCD_DATA3: track 0.00 -> 56.8 mm, vias 0 -> 2
- net LCD_DATA4: track 0.00 -> 56.4 mm
- net LCD_DATA5: track 0.00 -> 55.0 mm, vias 0 -> 2
- net LCD_DATA22: track 0.00 -> 54.9 mm, vias 0 -> 2
- net LCD_DATA19: track 0.00 -> 54.8 mm, vias 0 -> 2
- net LCD_DATA6: track 0.00 -> 54.1 mm, vias 0 -> 3
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- added copper zone on layer 1, net VIN
Other:
- outline, holes or cut-outs redrawn
- board text removed: "microphone"
