File: testBoard.sch (EAGLE design)
At the start: 19 parts, among them IC1 AM3358BZCZ100, IC3 LM317MABDT, J1 1040310811

Commit message: syncing edit
Parts:
- removed R5: 10ohm, rcl:R-EU_R0805W
- added IC5: REG1117, burr-brown:REG1117
- added JP1: (no value), pinhead:PINHD-1X2
- added U$2: 4_PIN_RESISTIVE_TOUCH, 4_pin_resistive_touch_pins:4_PIN_RESISTIVE_TOUCH
- R3, R4: value 10ohm -> 100ohm
Connections:
- removed net N$47: J1.VDD
- removed net N$48: J1.VSS
- removed net N$49: J1.DAT1
- removed net N$5: J1.CD/DAT3
- removed net N$52: R4.2, R5.2
- removed net N$53: R1.1, R4.1
- removed net N$54: R3.1
- removed net N$55: R1.2, R3.2
- removed net N$59: J1.DAT2
- removed net N$61: J1.CMD
- removed net N$62: J1.CLK
- removed net N$63: J1.DAT0
- removed net N$64: IC1.MMC0_DAT1
- removed net N$65: IC1.MMC0_DAT0
- removed net N$66: IC1.MMC0_CLK
- removed net N$67: IC1.MMC0_CMD
- removed net VO: C2.1, D2.C, D3.A, IC3.OUT
- new net N$37: IC3.OUT, R1.2
- new net N$9: IC3.ADJ
- new net SD_CLK: IC1.MMC0_CLK, J1.CLK
- new net SD_CMD: IC1.MMC0_CMD, J1.CMD
- new net SD_D0: IC1.MMC0_DAT0, J1.DAT0
- new net SD_D1: IC1.MMC0_DAT1, J1.DAT1
- new net SD_D2: IC1.MMC0_DAT2, J1.DAT2
- new net SD_D3: IC1.MMC0_DAT3, J1.CD/DAT3
- new net VIN_5: C2.1, D2.C, D3.A
- net GND: now also IC5.GND, J1.VSS, JP1.1, R3.1, R4.1
- net N$50: now also R1.1, R3.2, R4.2; no longer IC3.ADJ, R5.1
- net VIN: now also IC5.VIN, JP1.2
- net VIN_3.3: now also IC5.VOUT, J1.VDD
Other:
- note added: "3.3v power supply"
- note added: "TFT DISPLAY NHD-7.0-800480EF-ASXV#-T"
- note added: "memory IS42S16160G"
- note added: "processor AM3358BZCZ100"
- note added: "storage MOLEX 1040310811"
- note removed: "memory"
- note removed: "processor"
- note removed: "storage"
- moved on the sheet: R1, R2, R3, R4

Commit message: syncing edit
Connections:
- removed net N$45: IC1.DDR_DQS1
Changed lines of the file:
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@@
 <setting verticaltext="up"/>
 </settings>
-<grid distance="0.01" unitdist="mm" unit="mm" style="lines" multiple="1" display="yes" altdistance="0.01" altunitdist="inch" altunit="inch"/>
+<grid distance="0.1" unitdist="inch" unit="inch" style="lines" multiple="1" display="no" altdistance="0.01" altunitdist="inch" altunit="inch"/>
 <layers>
 <layer number="1" name="Top" color="4" fill="1" visible="no" active="no"/>
@@
 </segment>
 </net>
-<net name="N$45" class="0">
-<segment>
-<pinref part="IC1" gate="G$1" pin="DDR_DQS1"/>
-<wire x1="167.01" y1="385.767" x2="200.03" y2="385.767" width="0.1524" layer="91"/>
-</segment>
-</net>

Commit message: syncing edit
Parts:
- removed JP1: (no value), pinhead:PINHD-1X2
- added C10, C7: 1uf, rcl:C-EUC0805
- added C11, C8: 10uf, rcl:C-EUC0805
- added C6, C9: 0.01uf, rcl:C-EUC0805
- added D1, D4, D5, D6: 1n4002, diode:DIODE-DO-214AC
- added DISPLAY_POWER, PS1, PS2, PS3, PS4: (no value), pinhead:PINHD-1X2
- added IC2, IC4: LM317MABDT, v-reg:LM317MABDT
- added R10, R13, R16, R17, R5, R9: 10ohm, rcl:R-EU_R0805W
- added R11, R8: 1kohm, rcl:R-EU_R0805W
- added R12: 3.3kohm, rcl:R-EU_R0805W
- added R14, R19: 470ohm, rcl:R-EU_R0805W
- added R15: 100ohm, rcl:R-EU_R0805W
Connections:
- new net DISPLAY_POWER: DISPLAY-4.MS, DISPLAY_POWER.2
- new net N$38: R3.2, R4.2
- new net N$40: R12.1, R5.1
- new net N$41: R2.1, R3.1
- new net N$42: C8.1, D1.A, IC2.ADJ, R11.1, R12.2, R8.1
- new net N$43: R5.2, R9.2
- new net N$44: R10.1, R9.1
- new net N$45: R10.2, R13.2
- new net N$46: C11.1, D5.A, IC4.ADJ, R15.1, R19.2
- new net N$47: R14.1, R19.1
- new net N$48: R14.2, R16.2
- new net N$49: R16.1, R17.2
- new net VIN_1: D5.C, D6.A, IC4.OUT, R15.2
- new net VIN_12: C10.1
- new net VIN_9.6: C7.1
- net GND: now also C10.2, C11.2, C6.2, C7.2, C8.2, C9.2, PS1.1, PS2.1, PS3.1, PS4.1, R13.1, R17.1; no longer JP1.1, R2.1, R3.1
- net N$50: no longer R1.1, R2.2, R3.2, R4.2
- net N$9: now also R1.1, R2.2
- net VIN: now also C6.1, C9.1, D4.C, D6.C, IC2.IN, IC4.IN, PS1.2, PS2.2, PS3.2, PS4.2; no longer JP1.2
- net VIN_3.3: now also DISPLAY_POWER.1; no longer DISPLAY-4.MS
- net VIN_5: now also D1.C, D4.A, IC2.OUT, R11.2, R8.2
Other:
- note added: "12v power supply"
- note added: "9.6v power supply"
- note added: "Header pins"
- note added: "Led"

Commit message: Completed schematic for prototype 001
Parts:
- removed DISPLAY: XF2M-4015-1F, con-omron:XF2M-4015-1F
- removed IC5: REG1117, burr-brown:REG1117
- removed U$2: 4_PIN_RESISTIVE_TOUCH, 4_pin_resistive_touch_pins:4_PIN_RESISTIVE_TOUCH
- added J2: 54104-4031, 54104-4031:54104-4031
- added J3: 200529-0040, 200529-0040:200529-0040
Connections:
- removed net DISPLAY_EN: DISPLAY-35.MS
- removed net N$10: DISPLAY-5.MS
- removed net N$11: DISPLAY-6.MS
- removed net N$12: DISPLAY-7.MS
- removed net N$13: DISPLAY-8.MS
- removed net N$14: DISPLAY-9.MS
- removed net N$15: DISPLAY-10.MS
- removed net N$16: DISPLAY-11.MS
- removed net N$17: DISPLAY-12.MS
- removed net N$18: DISPLAY-13.MS
- removed net N$19: DISPLAY-14.MS
- removed net N$20: DISPLAY-15.MS
- removed net N$21: DISPLAY-16.MS
- removed net N$22: DISPLAY-17.MS
- removed net N$23: DISPLAY-18.MS
- removed net N$24: DISPLAY-19.MS
- removed net N$25: DISPLAY-20.MS
- removed net N$26: DISPLAY-21.MS
- removed net N$27: DISPLAY-22.MS
- removed net N$28: DISPLAY-23.MS
- removed net N$29: DISPLAY-24.MS
- removed net N$30: DISPLAY-25.MS
- removed net N$31: DISPLAY-26.MS
- removed net N$32: DISPLAY-27.MS
- removed net N$33: DISPLAY-28.MS
- removed net N$36: DISPLAY-31.MS
- removed net N$37: IC3.OUT, R1.2
- removed net N$39: DISPLAY-34.MS
- removed net N$6: DISPLAY-1.MSV
- removed net N$7: DISPLAY-2.MS
- new net LCD_AC_BIAS_EN: IC1.LCD_AC_BIAS_EN, J2.34
- new net LCD_DATA0: IC1.LCD_DATA0, J2.8
- new net LCD_DATA1: IC1.LCD_DATA1, J2.9
- new net LCD_DATA10: IC1.LCD_DATA10, J2.20
- new net LCD_DATA11: IC1.LCD_DATA11, J2.24
- new net LCD_DATA12: IC1.LCD_DATA12, J2.25
- new net LCD_DATA13: IC1.LCD_DATA13, J2.26
- new net LCD_DATA14: IC1.LCD_DATA14, J2.27
- new net LCD_DATA15: IC1.LCD_DATA15, J2.28
- new net LCD_DATA16: IC1.GPMC_AD15, J2.7
- new net LCD_DATA17: IC1.GPMC_AD14, J2.23
- new net LCD_DATA18: IC1.GPMC_AD13, J2.6
- new net LCD_DATA19: IC1.GPMC_AD12, J2.14
- new net LCD_DATA2: IC1.LCD_DATA2, J2.10
- new net LCD_DATA20: IC1.GPMC_AD11, J2.22
- new net LCD_DATA21: IC1.GPMC_AD10, J2.5
- new net LCD_DATA22: IC1.GPMC_AD9, J2.13
- new net LCD_DATA23: IC1.GPMC_AD8, J2.21
- new net LCD_DATA3: IC1.LCD_DATA3, J2.11
- new net LCD_DATA4: IC1.LCD_DATA4, J2.12
- new net LCD_DATA5: IC1.LCD_DATA5, J2.15
- new net LCD_DATA6: IC1.LCD_DATA6, J2.16
- new net LCD_DATA7: IC1.LCD_DATA7, J2.17
- new net LCD_DATA8: IC1.LCD_DATA8, J2.18
- new net LCD_DATA9: IC1.LCD_DATA9, J2.19
- new net LCD_MEMORY_CLK: IC1.GPMC_CLK
- new net LCD_TOUCH_XLEFT: IC1.AIN0, J3.1
- new net LCD_TOUCH_XRIGHT: IC1.AINI, J3.3
- new net LCD_TOUCH_YDOWN: IC1.AIN3, J3.2
- new net LCD_TOUCH_YUP: IC1.AIN2, J3.4
- net DISPLAY_POWER: now also J2.31; no longer DISPLAY-4.MS
- net GND: now also J2.1, J2.29, J2.3, J2.36; no longer DISPLAY-29.MS, DISPLAY-3.MS, DISPLAY-36.MS, IC5.GND
- net LCD_HSYNC: now also J2.32; no longer DISPLAY-32.MS
- net LCD_PCLK: now also J2.30; no longer DISPLAY-30.MS
- net LCD_VSYNC: now also J2.33; no longer DISPLAY-33.MS
- net VIN: no longer IC5.VIN
- net VIN_3.3: now also J2.4; no longer IC5.VOUT
- net VIN_9.6: now also J2.2

Commit message: checkpoint
Parts:
- removed R3, R4: 100ohm, rcl:R-EU_R0805W
- added C12, C15, C18: 0.01uf, rcl:C-EUC0805
- added C13, C16, C19: 1uf, rcl:C-EUC0805
- added C14, C17, C20: 10uf, rcl:C-EUC0805
- added D10, D11, D12, D7, D8, D9: 1n4002, diode:DIODE-DO-214AC
- added IC5, IC6, IC7: LM317MABDT, v-reg:LM317MABDT
- added J4: M50-3610542R, M50-3610542R:M50-3610542R
- added R18, R21, R23: 246ohm, rcl:R-EU_R0805W
- added R20, R22, R24: 150ohm, rcl:R-EU_R0805W
- R2: value 100ohm -> 30ohm
Connections:
- removed net N$38: R3.2, R4.2
- removed net N$41: R2.1, R3.1
- removed net N$50: C3.1, D2.A
- removed net VIN_1: D5.C, D6.A, IC4.OUT, R15.2
- new net JTAG_TCK: IC1.TCK, J4.4
- new net JTAG_TDI: IC1.TDI, J4.8
- new net JTAG_TDO: IC1.TDO, J4.6
- new net JTAG_TEST_RESET_NTRST: IC1.TRSTN, J4.9
- new net JTAG_TMS: IC1.TMS, J4.2
- new net N$10: C20.1, D11.A, IC7.ADJ, R23.2, R24.1
- new net N$6: C14.1, D7.A, IC5.ADJ, R18.2, R20.1
- new net N$7: C17.1, D9.A, IC6.ADJ, R21.2, R22.1
- new net NRESET_IN_OUT_AM3358: IC1.WARMRSTN, J4.10
- net GND: now also C12.2, C13.2, C14.2, C15.2, C16.2, C17.2, C18.2, C19.2, C20.2, J4.3, J4.5, R18.1, R2.1, R21.1, R23.1; no longer R4.1
- net N$9: now also C3.1, D2.A
- net VIN: now also C12.1, C15.1, C18.1, D10.C, D12.C, D8.C, IC5.IN, IC6.IN, IC7.IN
- net VIN_12: now also D5.C, D6.A, IC4.OUT, R15.2
- net VIN_3.3: now also C13.1, C16.1, C19.1, D10.A, D11.C, D12.A, D7.C, D8.A, D9.C, IC5.OUT, IC6.OUT, IC7.OUT, J4.1, R20.2, R22.2, R24.2
- net VIN_5: now also IC3.OUT, R1.2; no longer D1.C, D4.A, IC2.OUT, R11.2, R8.2
- net VIN_9.6: now also D1.C, D4.A, IC2.OUT, R11.2, R8.2
Other:
- note added: "3.3V, 500mA"
- note added: "debugger"
- moved on the sheet: C10, C11, C9, D5, D6, IC4, R15, R2
